Commit message: added inertial properties

File: my_robot_description/urdf/common_properties.xacro (robot description, xacro)
@@ -10,3 +10,30 @@
         <color rgba="0 0 0.5 1" />
     </material>
+    <xacro:macro name="box_inertial" params="m l w h xyz rpy">
+        <inertial>
+            <origin xyz="${xyz}" rpy="${rpy}" />
+            <mass value="${m}" />
+            <inertia ixx="${(m/12)*(l*l + h*h)}" ixy="0" ixz="0"
+            iyy="${(m/12)*(w*w + l*l)}" iyz="0"
+            izz="${(m/12)*(w*w + h*h)}" />
+        </inertial>
+    </xacro:macro>
+    <xacro:macro name="wheel_inertial" params="m r l xyz rpy">
+        <inertial>
+            <origin xyz="${xyz}" rpy="${rpy}" />
+            <mass value="${m}" />
+            <inertia ixx="${(m/12)*(3*r*r + l*l)}" ixy="0" ixz="0"
+            iyy="${(m/12)*(3*r*r + l*l)}" iyz="0"
+            izz="${(m/2)*r*r}" />
+        </inertial>
+    </xacro:macro>
+    <xacro:macro name="caster_wheel_inertial" params="m r xyz rpy">
+        <inertial>
+            <origin xyz="${xyz}" rpy="${rpy}" />
+            <mass value="${m}" />
+            <inertia ixx="${(2*m/5)*(r*r)}" ixy="0" ixz="0"
+            iyy="${(2*m/5)*(r*r)}" iyz="0"
+            izz="${(2*m/5)*(r*r)}" />
+        </inertial>
+    </xacro:macro>
 </robot>

File: my_robot_description/urdf/mobile_base.xacro (robot description, xacro)
@@ -14,4 +14,6 @@
             <material name="green" />
         </visual>
+        <xacro:box_inertial m="5.0" l="${base_length}"
+        w="${base_width}" h="${base_height}" xyz="0 0 ${base_height / 2.0}" rpy="0 0 0" />
     </link>
     <xacro:macro name="wheel_link" params="prefix">
@@ -24,4 +26,6 @@
                 <material name="grey" />
             </visual>
+            <xacro:wheel_inertial m="1.0" r="${wheel_radius}" l="${wheel_length}" xyz="0 0 0"
+            rpy="${pi / 2.0} 0 0" />
         </link>
     </xacro:macro>
@@ -31,9 +35,11 @@
         <visual>
             <geometry>
-                <sphere radius="0.05" />
+                <sphere radius="${wheel_length}" />
             </geometry>
             <origin xyz="0 0 ${-wheel_radius / 2.0}" rpy="0 0 0" />
             <material name="grey" />
         </visual>
+        <xacro:caster_wheel_inertial m="0.5" r="${wheel_length}"
+        xyz="0 0 ${-wheel_radius / 2.0}" rpy="0 0 0" />
     </link>
     <link name="base_footprint" />

Commit message: completed the robotic arm with all joints intact

File: my_robot_description/urdf/common_properties.xacro (robot description, xacro)
@@ -9,4 +9,10 @@
     <material name="blue">
         <color rgba="0 0 0.5 1" />
+    </material>
+    <material name="orange">
+        <color rgba="1 0.647 0 1" />
+    </material>
+    <material name="yellow">
+        <color rgba="1 1 0 1" />
     </material>
     <xacro:macro name="box_inertial" params="m l w h xyz rpy">
