Commit message: added gazebo launch file

File: my_robot_description/urdf/mobile_base.xacro (robot description, xacro)
@@ -14,4 +14,10 @@
             <material name="green" />
         </visual>
+        <collision>
+            <geometry>
+                <box size="${base_length} ${base_width} ${base_height}" />
+            </geometry>
+            <origin xyz="0 0 ${base_height / 2.0}" rpy="0 0 0" />
+        </collision>
         <xacro:box_inertial m="5.0" l="${base_length}"
         w="${base_width}" h="${base_height}" xyz="0 0 ${base_height / 2.0}" rpy="0 0 0" />
@@ -26,4 +32,10 @@
                 <material name="grey" />
             </visual>
+            <collision>
+                <geometry>
+                    <cylinder radius="${wheel_radius}" length="${wheel_length}" />
+                </geometry>
+                <origin xyz="0 0 0" rpy="${pi / 2.0} 0 0" />
+            </collision>
             <xacro:wheel_inertial m="1.0" r="${wheel_radius}" l="${wheel_length}" xyz="0 0 0"
             rpy="${pi / 2.0} 0 0" />
@@ -40,4 +52,10 @@
             <material name="grey" />
         </visual>
+        <collision>
+            <geometry>
+                <sphere radius="${wheel_length}" />
+            </geometry>
+            <origin xyz="0 0 ${-wheel_radius / 2.0}" rpy="0 0 0" />
+        </collision>
         <xacro:caster_wheel_inertial m="0.5" r="${wheel_length}"
         xyz="0 0 ${-wheel_radius / 2.0}" rpy="0 0 0" />

Commit message: joined the robotic arm with the mobile base

File: my_robot_description/urdf/mobile_base.xacro (robot description, xacro)
@@ -6,4 +6,5 @@
     <xacro:property name="wheel_radius" value="0.1" />
     <xacro:property name="wheel_length" value="0.05" />
+    <xacro:include filename="robotic_arm.xacro" />
     <link name="base_link">
         <visual>
@@ -84,3 +85,8 @@
         <origin xyz="0 0 ${wheel_radius}" rpy="0 0 0" />
     </joint>
+    <joint name="base_arm_base_joint" type="fixed">
+        <parent link="base_link" />
+        <child link="arm_base_link" />
+        <origin xyz="0 0 ${base_height}" rpy="0 0 0" />
+    </joint>
 </robot>

File: my_robot_description/urdf/my_robot.urdf.xacro (robot description, xacro)
@@ -3,4 +3,5 @@
     <xacro:include filename="common_properties.xacro" />
     <xacro:include filename="mobile_base.xacro" />
+    <xacro:include filename="robot_arm_gazebo.xacro" />
     <xacro:include filename="mobile_base_gazebo.xacro" />
     <xacro:include filename="camera.xacro" />

File: my_robot_description/urdf/robotic_arm.xacro (robot description, xacro)
@@ -1,4 +1,4 @@
 <?xml version="1.0"?>
-<robot name="robotic_arm" xmlns:xacro="http://www.ros.org/wiki/xacro">
+<robot xmlns:xacro="http://www.ros.org/wiki/xacro">
     <xacro:property name="arm_base_length" value="0.1" />
     <xacro:property name="arm_base_width" value="0.1" />
@@ -6,5 +6,4 @@
     <xacro:property name="common_arm_radius" value="0.02" />
     <xacro:property name="common_arm_length" value="0.3" />
-    <xacro:include filename="common_properties.xacro" />
     <link name="arm_base_link">
         <visual>
@@ -12,5 +11,5 @@
                 <box size="${arm_base_length} ${arm_base_width} ${arm_base_height}" />
             </geometry>
-            <origin xyz="0 0 0" rpy="0 0 0" />
+            <origin xyz="0 0 ${arm_base_height/2}" rpy="0 0 0" />
             <material name="orange" />
         </visual>

Commit message: added final touches to the complete robot

File: my_robot_description/urdf/mobile_base.xacro (robot description, xacro)
@@ -88,5 +88,5 @@
         <parent link="base_link" />
         <child link="arm_base_link" />
-        <origin xyz="0 0 ${base_height}" rpy="0 0 0" />
+        <origin xyz="${base_length/3} 0 ${base_height}" rpy="0 0 0" />
     </joint>
 </robot>

File: my_robot_description/urdf/mobile_base_gazebo.xacro (robot description, xacro)
@@ -1,4 +1,5 @@
 <?xml version="1.0"?>
 <robot xmlns:xacro="http://www.ros.org/wiki/xacro">
+    <xacro:include filename="robot_arm_gazebo.xacro" />
     <gazebo reference="base_link">
         <material>Gazebo/Blue</material>

File: my_robot_description/urdf/my_robot.urdf.xacro (robot description, xacro)
@@ -3,5 +3,4 @@
     <xacro:include filename="common_properties.xacro" />
     <xacro:include filename="mobile_base.xacro" />
-    <xacro:include filename="robot_arm_gazebo.xacro" />
     <xacro:include filename="mobile_base_gazebo.xacro" />
     <xacro:include filename="camera.xacro" />

File: my_robot_description/urdf/robot_arm_gazebo.xacro (robot description, xacro)
@@ -11,5 +11,5 @@
     </gazebo>
     <gazebo>
-        <plugin name="gazebo_ros_joint_state_publisher"
+        <plugin name="joint_state_publisher"
         filename="libgazebo_ros_joint_state_publisher.so">
             <!-- Update rate in Hertz -->
@@ -21,5 +21,5 @@
     </gazebo>
     <gazebo>
-        <plugin name="gazebo_ros_joint_pose_trajectory"
+        <plugin name="joint_pose_trajectory"
         filename="libgazebo_ros_joint_pose_trajectory.so">
         <!-- Update rate in Hz -->

File: my_robot_description/urdf/robotic_arm.xacro (robot description, xacro)
@@ -50,5 +50,5 @@
         <limit lower="0" upper="${pi/2}" effort="100" velocity="100" />
         <dynamic friction="0.05" damping="0.1" />
-        <axis xyz="0 0 1"/>
+        <axis xyz="0 1 0"/>
     </joint>
     <joint name="forearm_hand_joint" type="revolute">
@@ -58,5 +58,5 @@
         <limit lower="0" upper="${pi/2}" effort="100" velocity="100" />
         <dynamic friction="0.05" damping="0.1" />
-        <axis xyz="0 0 1"/>
+        <axis xyz="0 1 0"/>
     </joint>
 </robot>
